File: lab4/exercise 1/exercise 1.kicad_sch (KiCad schematic)
At the start: 6 parts, among them J1 Conn_01x02_Male, SW1 SW_SPDT

Commit message: lab6
Parts:
- C1: footprint (none) -> Capacitor_THT:C_Radial_D5.0mm_H5.0mm_P2.00mm
- D1: footprint (none) -> LED_THT:LED_D5.0mm
- J1: footprint (none) -> Connector_JST:JST_PH_B2B-PH-K_1x02_P2.00mm_Vertical
- R1, R2: footprint (none) -> Resistor_THT:R_Axial_DIN0516_L15.5mm_D5.0mm_P20.32mm_Horizontal
- SW1: footprint (none) -> Button_Switch_THT:SW_E-Switch_EG1224_SPDT_Angled
Changed lines of the file:
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@@
       (effects (font (size 1.27 1.27)) (justify left))
     )
-    (property "Footprint" "" (id 2) (at 191.4652 87.63 0)
+    (property "Footprint" "Capacitor_THT:C_Radial_D5.0mm_H5.0mm_P2.00mm" (id 2) (at 191.4652 87.63 0)
       (effects (font (size 1.27 1.27)) hide)
     )
@@
       (effects (font (size 1.27 1.27)) (justify left))
     )
-    (property "Footprint" "" (id 2) (at 216.662 72.39 90)
+    (property "Footprint" "Resistor_THT:R_Axial_DIN0516_L15.5mm_D5.0mm_P20.32mm_Horizontal" (id 2) (at 216.662 72.39 90)
       (effects (font (size 1.27 1.27)) hide)
     )
@@
     (property "Reference" "SW1" (id 0) (at 170.18 58.42 0))
     (property "Value" "SW_SPDT" (id 1) (at 170.18 60.96 0))
-    (property "Footprint" "" (id 2) (at 170.18 66.04 0)
+    (property "Footprint" "Button_Switch_THT:SW_E-Switch_EG1224_SPDT_Angled" (id 2) (at 170.18 66.04 0)
       (effects (font (size 1.27 1.27)) hide)
     )
@@
     (property "Reference" "D1" (id 0) (at 218.1225 95.25 0))
     (property "Value" "LED" (id 1) (at 218.1225 97.79 0))
-    (property "Footprint" "" (id 2) (at 219.71 101.6 0)
+    (property "Footprint" "LED_THT:LED_D5.0mm" (id 2) (at 219.71 101.6 0)
       (effects (font (size 1.27 1.27)) hide)
     )
@@
     (property "Reference" "J1" (id 0) (at 128.905 80.01 0))
     (property "Value" "Conn_01x02_Male" (id 1) (at 128.905 82.55 0))
-    (property "Footprint" "" (id 2) (at 128.27 85.09 0)
+    (property "Footprint" "Connector_JST:JST_PH_B2B-PH-K_1x02_P2.00mm_Vertical" (id 2) (at 128.27 85.09 0)
       (effects (font (size 1.27 1.27)) hide)
     )
@@
   (symbol (lib_id "Device:R") (at 139.7 66.04 90) (unit 1)
     (in_bom yes) (on_board yes) (fields_autoplaced)
-    (property "Reference" "R2" (id 0) (at 138.4299 63.5 0)
-      (effects (font (size 1.27 1.27)) (justify left))
-    )
-    (property "Value" "2.2k" (id 1) (at 140.9699 63.5 0)
-      (effects (font (size 1.27 1.27)) (justify left))
-    )
-    (property "Footprint" "" (id 2) (at 139.7 67.818 90)
+    (property "Reference" "R2" (id 0) (at 139.7 59.69 90))
+    (property "Value" "2.2k" (id 1) (at 139.7 62.23 90))
+    (property "Footprint" "Resistor_THT:R_Axial_DIN0516_L15.5mm_D5.0mm_P20.32mm_Horizontal" (id 2) (at 139.7 67.818 90)
       (effects (font (size 1.27 1.27)) hide)
     )
@@
   (symbol_instances
     (path "/0676efd1-2736-48e3-b8af-64917230e4e2"
-      (reference "C1") (unit 1) (value "4.7µF") (footprint "")
+      (reference "C1") (unit 1) (value "4.7µF") (footprint "Capacitor_THT:C_Radial_D5.0mm_H5.0mm_P2.00mm")
     )
     (path "/5d00ca34-9f9a-4dcb-b9c7-93127f285e00"
-      (reference "D1") (unit 1) (value "LED") (footprint "")
+      (reference "D1") (unit 1) (value "LED") (footprint "LED_THT:LED_D5.0mm")
     )
     (path "/70443a09-7056-4048-b2d3-fcf9b633ad2c"
-      (reference "J1") (unit 1) (value "Conn_01x02_Male") (footprint "")
+      (reference "J1") (unit 1) (value "Conn_01x02_Male") (footprint "Connector_JST:JST_PH_B2B-PH-K_1x02_P2.00mm_Vertical")
     )
     (path "/41b4632d-3ec0-4a0f-a6b4-cf7a029d5fdc"
-      (reference "R1") (unit 1) (value "20k") (footprint "")
+      (reference "R1") (unit 1) (value "20k") (footprint "Resistor_THT:R_Axial_DIN0516_L15.5mm_D5.0mm_P20.32mm_Horizontal")
     )
     (path "/e2d2cbb6-7755-423f-8b74-519d20a632bc"
-      (reference "R2") (unit 1) (value "2.2k") (footprint "")
+      (reference "R2") (unit 1) (value "2.2k") (footprint "Resistor_THT:R_Axial_DIN0516_L15.5mm_D5.0mm_P20.32mm_Horizontal")
     )
     (path "/52b18cb1-42e7-4bf8-9972-000f04f6515a"
-      (reference "SW1") (unit 1) (value "SW_SPDT") (footprint "")
+      (reference "SW1") (unit 1) (value "SW_SPDT") (footprint "Button_Switch_THT:SW_E-Switch_EG1224_SPDT_Angled")
     )
   )
